File: 68k.kicad_sch (KiCad schematic)
At the start: 33 parts, among them J1 Conn_01x08_Socket, J2 Conn_01x08_Socket, J3 Conn_01x06_Socket, Q1 BC547, Q2 BC547, SW1 Reset button, U1 MC68000P, U10 MAX1232CPA, U11 74LS161, U12 74HCT00, U2 27C020, U3 27C020, U4 AS6C4008-55PCN, U5 AS6C4008-55PCN, U6 MC68A21, U7 MC68A40, U8 MC68A50, U9 PCF8584, Y1 8.0 MHz, Y2 1.8432 MHz

Commit message: Project: 68000 system architecture
Parts:
- removed U12: 74HCT00, symbol 74xx:74HCT00
- added D3: Power/strobe OK, symbol Device:LED_Small
- added J4, J5: Conn_01x02_Socket, symbol Connector:Conn_01x02_Socket
- added R10, R11, R12, R13, R9: 10k, symbol Device:R
- added R6: 2.2k, symbol Device:R
- added R7, R8: 4.7k, symbol Device:R
- added SW2: Abort button, symbol Switch:SW_Push
- added U12: 74LS03, symbol 74xx:74LS03
- added U13: GAL16V8, symbol Logic_Programmable:GAL16V8
- added U14: 74LS161, symbol 74xx:74LS161
- added U15: 74LS32, symbol 74xx:74LS32
- added U16: 74LS04, symbol 74xx:74LS04
- added U17: 74LS22, symbol 74xx:74LS22
- added U18: 74HC238, symbol 74xx:74HC238
- added U19: 74LS148, symbol 74xx:74LS148
- added U20: PCF8563T, Package_SO:SOIC-8_3.9x4.9mm_P1.27mm, symbol Timer_RTC:PCF8563T
- added Y3: Crystal, symbol Device:Crystal
Connections:
- net +5V: now also U6.22 (CS0), U8.10 (CS1), R10.1, R11.1, R12.2, R13.2, R6.1, R7.2, R8.2, R9.1, U12.14 (VCC), U13.20 (V_{CC}), U14.1 (~{MR}), U14.10 (CET), U14.16 (VCC), U14.6 (D3), U15.14 (VCC), U16.14 (VCC), U17.14 (VCC), U18.16 (VCC), U18.5 (~{E2}), U18.6 (E3), U19.10 (IO), U19.16 (VCC), U20.8 (VDD); no longer U2.31 (~{PGM}), U3.31 (~{PGM})
- net A1: now also U6.36 (RS0), U7.10 (RS0), U8.11 (RS), U9.6 (A0)
- net A16: now also U18.1 (A0)
- net A17: now also U18.2 (A1)
- net A18: now also U12.2, U13.6 (I_{5}), U18.3 (A2)
- net A19: now also U13.5 (I_{4})
- net A2: now also U6.35 (RS1), U7.11 (RS1)
- net A20: now also U13.4 (I_{3})
- net A21: now also U13.3 (I_{2})
- net A22: now also U13.2 (I_{1})
- net A23: now also U13.1 (I_{0})
- net A3: now also U7.12 (RS2)
- net Baudrate: now also U12.6
- net DTACK: now also U16.8; no longer U10.7 (~{ST})
- net GND: now also D3.1 (K), SW2.2, U12.7 (GND), U13.10 (GND), U14.3 (D0), U14.4 (D1), U14.5 (D2), U14.8 (GND), U15.7 (GND), U16.7 (GND), U17.7 (GND), U18.8 (GND), U19.5 (EI), U19.8 (GND), U20.4 (VSS); no longer J3.5 (Pin_5), U8.5 (~{RTS})
- net RW: now also U9.18 (~{WR}), U13.9 (I_{8}), U15.10, U15.13
- net Reset: now also U9.19 (~{RST})
- net VMA: now also U6.23 (~{CS2}), U7.15 (~{CS0}), U8.9 (CS2)
- net X0: now also U9.1 (CLK), U14.2 (CP)
- net SRAM CE: now reaches U5.22 (CE#)
- net SRAM CE: now also U4.22 (CE#), U13.15 (F_{3}), U17.10
- net SRAMH OE: now reaches U5.24 (OE#)
- net SRAMH OE: now also U15.6
- net SRAMH WE: now reaches U5.29 (WE#)
- net SRAMH WE: now also U15.8
- net 84 DTACK: now reaches U9.16 (~{RD})
- net 84 DTACK: now also U17.13
- net 84 CE: now reaches U9.17 (~{CS})
- net 84 CE: now also U16.12
- net SDA: now reaches U9.2 (SDA)
- net SDA: now also R7.1, U20.5 (SDA)
- net SCL: now reaches U9.3 (SCL)
- net SCL: now also R8.1, U20.6 (SCL)
- net 84 IRQ: now reaches U9.5 (~{INT})
- net 84 IRQ: now also U19.12 (I2)
- net 40 CE: now reaches U7.16 (CS1)
- net 40 CE: now also U18.10 (Y5)
- net 40 IRQ: now reaches U7.9 (~{IRQ})
- net 40 IRQ: now also U19.3 (I6)
- net EEPROM CE: now reaches U2.22 (~{CE})
- net EEPROM CE: now also U3.22 (~{CE}), U13.16 (F_{4}), U17.9
- net LDS: now reaches U2.24 (~{OE})
- net LDS: now also U1.8 (~{LDS}), U15.1, U15.12
- net UDS: now reaches U3.24 (~{OE})
- net UDS: now also U1.7 (~{UDS}), U15.4, U15.9
- net SRAML OE: now reaches U4.24 (OE#)
- net SRAML OE: now also U15.3
- net SRAML WE: now reaches U4.29 (WE#)
- net SRAML WE: now also U15.11
- net 50 IRQ: now reaches U8.7 (~{IRQ})
- net 50 IRQ: now also U19.1 (I4)
- net 50 CE: now reaches U8.8 (CS0)
- net 50 CE: now also U18.9 (Y6)
- net at U6.18 (CB1): now also J5.1 (Pin_1)
- net at U6.19 (CB2): now also J5.2 (Pin_2)
- net 21 CE: now reaches U6.24 (CS1)
- net 21 CE: now also U18.11 (Y4)
- net 21B IRQ: now reaches U6.37 (~{IRQB})
- net 21B IRQ: now also U19.13 (I3)
- net 21A IRQ: now reaches U6.38 (~{IRQA})
- net 21A IRQ: now also U19.11 (I1)
- net at U6.39 (CA2): now also J4.2 (Pin_2)
- net at U6.40 (CA1): now also J4.1 (Pin_1)
- net at U11.12 (Q2): now also U12.4
- net at U11.11 (Q3): now also U12.5
- net VPA: now reaches U1.21 (~{VPA})
- net VPA: now also R12.1, U12.3, U17.6
- net BERR: now reaches U1.22 (~{BERR})
- net BERR: now also U13.14 (F_{2})
- net IPL2: now reaches U1.23 (~{IPL2})
- net IPL2: now also U19.6 (S2)
- net IPL1: now reaches U1.24 (~{IPL1})
- net IPL1: now also U19.7 (S1)
- net IPL0: now reaches U1.25 (~{IPL0})
- net IPL0: now also U19.9 (S0)
- net FC2: now reaches U1.26 (FC2)
- net FC2: now also U13.8 (I_{7}), U17.4
- net FC1: now reaches U1.27 (FC1)
- net FC1: now also U17.2
- net FC0: now reaches U1.28 (FC0)
- net FC0: now also U17.1
- net AS: now reaches U1.6 (~{AS})
- net AS: now also U13.7 (I_{6}), U16.5
- net Force Halt: now reaches U10.6 (~{RST})
- net Force Halt: now also D3.2 (A), R6.2
- new net: U20.1 (OSCI), Y3.1
- new net: U20.2 (OSCO), Y3.2
- new net: R10.2, U16.9, U17.8
- new net: R11.2, U17.12
- new net: U16.6, U17.5
- new net: U16.13, U18.15 (Y0)
- new net: J3.5 (Pin_5), U8.5 (~{RTS})
- new net: R9.2, U13.13 (F_{1})
- new net 83 IRQ: U19.2 (I5), U20.3 (~{INT})
- new net Abort: R13.1, SW2.1, U19.4 (I7)
- new net E0: U13.18 (F_{6})
- new net IO CE: U12.1, U13.19 (F_{7}), U18.4 (~{E1})
- new net RD: U13.17 (F_{5}), U15.2, U15.5
- new net TO: U13.11 (I_{9}), U14.11 (Q3), U14.7 (CEP)
- new net TR: U13.12 (F_{0}), U14.9 (~{PE})
- new net Watchdog: U10.7 (~{ST}), U18.7 (Y7)
- no-connect marks 5 -> 17
Other:
- note added: "Address Decoding And Bus Timeout"
- note added: "Frequency Generator Circuit"
- note added: "I/O Decoder"
- note added: "I2^C Bus"
- note added: "Interrupt Encoder"
- note removed: "Clock Generator Circuit"
- moved on the sheet: C1, C2, C3, C4, C5, C6, D1, D2, Q1, Q2, R1, R2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

Commit message: Project: add I/O pins, fix wrong connections
Parts:
- added C7, C8: 0.1µF, symbol Device:C_Small
- added C9: 24pF, symbol Device:C_Small
- added J10: BERR, symbol Connector:Conn_01x01_Socket
- added J11: Stretch Cycle, symbol Connector:Conn_01x01_Socket
- added J12: Expansion Slot 0, symbol Connector:Conn_01x01_Socket
- added J13: Control Output, symbol Connector:Conn_01x07_Socket
- added J14: Address Bus, symbol Connector:Conn_01x23_Socket
- added J15: Lower Data Bus, symbol Connector:Conn_01x08_Socket
- added J16: Upper Data Bus, symbol Connector:Conn_01x08_Socket
- added J6: Timer 1, symbol Connector:Conn_01x03_Socket
- added J7: Timer 2, symbol Connector:Conn_01x03_Socket
- added J8: Timer 3, symbol Connector:Conn_01x03_Socket
- added J9: DTACK, symbol Connector:Conn_01x01_Socket
- added R14, R15: 10k, symbol Device:R
- added unit 5 of U12
- added unit 1 of U12
- added unit 1 of U15
- added unit 4 of U15
- added unit 3 of U15
- added unit 5 of U15
- added unit 6 of U16
- added unit 7 of U16
- added unit 3 of U17
- added unit 1 of U17
- J1: value Conn_01x08_Socket -> PORT A
- J2: value Conn_01x08_Socket -> PORT B
- J3: value Conn_01x06_Socket -> Serial I/O
- J4: value Conn_01x02_Socket -> CTRL A
- J5: value Conn_01x02_Socket -> CTRL B
Connections:
- net +5V: now also C7.2, C8.2, R14.1, R15.1, U12.14 (VCC), U15.14 (VCC), U16.14 (VCC), U17.14 (VCC); no longer U12.14 (VCC), U14.10 (CET), U15.14 (VCC), U16.14 (VCC), U17.14 (VCC), U18.5 (~{E2}), U18.6 (E3)
- net 84 CE: now also U16.12; no longer U16.12
- net A1: now also J14.1 (Pin_1)
- net A10: now also J14.10 (Pin_10)
- net A11: now also J14.11 (Pin_11)
- net A12: now also J14.12 (Pin_12)
- net A13: now also J14.13 (Pin_13)
- net A14: now also J14.14 (Pin_14)
- net A15: now also J14.15 (Pin_15)
- net A16: now also J14.16 (Pin_16)
- net A17: now also J14.17 (Pin_17)
- net A18: now also J14.18 (Pin_18), U12.2; no longer U12.2
- net A19: now also J14.19 (Pin_19)
- net A2: now also J14.2 (Pin_2)
- net A20: now also J14.20 (Pin_20)
- net A21: now also J14.21 (Pin_21)
- net A22: now also J14.22 (Pin_22)
- net A23: now also J14.23 (Pin_23)
- net A3: now also J14.3 (Pin_3)
- net A4: now also J14.4 (Pin_4)
- net A5: now also J14.5 (Pin_5)
- net A6: now also J14.6 (Pin_6)
- net A7: now also J14.7 (Pin_7)
- net A8: now also J14.8 (Pin_8)
- net A9: now also J14.9 (Pin_9)
- net AS: now also J13.2 (Pin_2)
- net Baudrate: now also R15.2
- net DA0: now also J15.1 (Pin_1)
- net DA1: now also J15.2 (Pin_2)
- net DA2: now also J15.3 (Pin_3)
- net DA3: now also J15.4 (Pin_4)
- net DA4: now also J15.5 (Pin_5)
- net DA5: now also J15.6 (Pin_6)
- net DA6: now also J15.7 (Pin_7)
- net DA7: now also J15.8 (Pin_8)
- net DB0: now also J16.1 (Pin_1)
- net DB1: now also J16.2 (Pin_2)
- net DB2: now also J16.3 (Pin_3)
- net DB3: now also J16.4 (Pin_4)
- net DB4: now also J16.5 (Pin_5)
- net DB5: now also J16.6 (Pin_6)
- net DB6: now also J16.7 (Pin_7)
- net DB7: now also J16.8 (Pin_8)
- net FC0: now also U17.1; no longer U17.1
- net FC1: now also U17.2; no longer U17.2
- net FC2: now also J13.6 (Pin_6), U17.4; no longer U17.4
- net GND: now also U18.4 (~{E1}), U18.5 (~{E2}), C7.1, C8.1, C9.1, U12.7 (GND), U15.7 (GND), U16.7 (GND), U17.7 (GND); no longer U12.7 (GND), U15.7 (GND), U16.7 (GND), U17.7 (GND)
- net IO CE: now also U18.6 (E3), U12.1; no longer U12.1, U18.4 (~{E1})
- net LDS: now also J13.5 (Pin_5), U15.1, U15.12; no longer U15.1, U15.12
- net RD: now also U15.2; no longer U15.2
- net RW: now also J13.3 (Pin_3), U15.10, U15.13; no longer U15.10, U15.13
- net Reset: now also J13.7 (Pin_7)
- net SRAMH WE: now also U15.8; no longer U15.8
- net SRAML OE: now also U15.3; no longer U15.3
- net SRAML WE: now also U15.11; no longer U15.11
- net UDS: now also J13.4 (Pin_4), U15.9; no longer U15.9
- net VPA: now also U12.3, U17.6; no longer U12.3, U17.6
- net X0: now also J13.1 (Pin_1)
- net at U20.2 (OSCO), Y3.2: now also C9.2
- net at U7.2 (~{G2}): now also J7.1 (Pin_1)
- net at U7.26 (~{G1}): now also J6.1 (Pin_1)
- net at U7.27 (O1): now also J6.3 (Pin_3)
- net at U7.28 (~{C1}): now also J6.2 (Pin_2)
- net at U7.3 (O2): now also J7.3 (Pin_3)
- net at U7.4 (~{C2}): now also J7.2 (Pin_2)
- net at U7.5 (~{G3}): now also J8.1 (Pin_1)
- net at U7.6 (O3): now also J8.3 (Pin_3)
- net at U7.7 (~{C3}): now also J8.2 (Pin_2)
- net at R11.2, U17.12: now also J9.1 (Pin_1)
- net at U16.6: now also U17.5; no longer U17.5
- net at U18.15 (Y0): now also U16.13; no longer U16.13
- net at R9.2, U13.13 (F_{1}): now also J10.1 (Pin_1)
- net E0: no longer names the net of U13.18 (F_{6})
- net E0: now also J12.1 (Pin_1)
- new net: J11.1 (Pin_1), R14.2, U14.10 (CET)
Other:
- moved on the sheet: C1, C2, C3, C4, C5, C6, D1, D3, J3, R1, R10, R11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
